Commit message: fix

File: src/robot_description/urdf/gazebo_plugins.xacro (robot description, xacro)
@@ -7,6 +7,6 @@
       <left_joint>left_wheel_joint</left_joint>
       <right_joint>right_wheel_joint</right_joint>
-      <wheel_separation>0.35</wheel_separation>
-      <wheel_radius>0.07</wheel_radius>
+      <wheel_separation>0.38</wheel_separation>
+      <wheel_radius>0.05</wheel_radius>
       <odom_publish_frequency>20</odom_publish_frequency>
       <topic>/cmd_vel</topic>
@@ -36,11 +36,25 @@
     </plugin>
   </gazebo>
-  <!-- ===================== CASTER FRICTION ===================== -->
-  <!-- Zero friction so the fixed sphere slides freely without fighting the drive wheels -->
+  <!-- ===================== WHEEL / CASTER SURFACE PHYSICS ============ -->
+  <gazebo reference="left_wheel">
+    <mu1>1.5</mu1>
+    <mu2>1.5</mu2>
+    <kp>1000000.0</kp>
+    <kd>10.0</kd>
+    <minDepth>0.001</minDepth>
+  </gazebo>
+  <gazebo reference="right_wheel">
+    <mu1>1.5</mu1>
+    <mu2>1.5</mu2>
+    <kp>1000000.0</kp>
+    <kd>10.0</kd>
+    <minDepth>0.001</minDepth>
+  </gazebo>
   <gazebo reference="caster_wheel">
-    <mu1>0.0</mu1>
-    <mu2>0.0</mu2>
+    <mu1>0.01</mu1>
+    <mu2>0.01</mu2>
     <kp>1000000.0</kp>
-    <kd>100.0</kd>
+    <kd>10.0</kd>
+    <minDepth>0.001</minDepth>
   </gazebo>
   <!-- ===================== LIDAR ===================== -->

File: src/robot_description/urdf/service_robot.urdf.xacro (robot description, xacro)
@@ -3,34 +3,16 @@
   <xacro:include filename="$(find robot_description)/urdf/gazebo_plugins.xacro"/>
   <!-- ===================== PROPERTIES ===================== -->
-  <!--
-    Layout inspired by the Gazebo tutorial car:
-      - Chassis elevated so its bottom is at wheel-axle height
-      - Drive wheels mounted at the REAR of the chassis
-      - Front ball-caster provides the third contact point
-  -->
-  <xacro:property name="base_length"   value="0.45"/>
-  <xacro:property name="base_width"    value="0.30"/>
-  <xacro:property name="base_height"   value="0.15"/>
-  <xacro:property name="wheel_radius"  value="0.07"/>
-  <xacro:property name="wheel_width"   value="0.05"/>
-  <xacro:property name="caster_radius" value="0.035"/>   <!-- wheel_radius / 2 -->
-  <!-- drive wheels are offset 12 cm toward the rear of the chassis -->
-  <xacro:property name="wheel_x"       value="-0.12"/>
-  <!-- derived: wheel separation = base_width + wheel_width -->
-  <xacro:property name="wheel_sep"     value="${base_width + wheel_width}"/>  <!-- 0.35 m -->
-  <!-- ===================== BASE FOOTPRINT ===================== -->
+  <xacro:property name="base_length" value="0.4"/>
+  <xacro:property name="base_width" value="0.3"/>
+  <xacro:property name="base_height" value="0.15"/>
+  <xacro:property name="wheel_radius" value="0.05"/>
+  <xacro:property name="wheel_width" value="0.04"/>
+  <!-- ===================== BASE LINK ===================== -->
   <link name="base_footprint"/>
-  <!--
-    Chassis centre must sit at  wheel_radius + base_height/2  above base_footprint
-    so that the chassis bottom is flush with the drive-wheel axle plane and the
-    wheels just touch the ground (z = 0).
-      wheel_radius=0.07, base_height/2=0.075  →  joint z = 0.145
-  -->
   <joint name="base_footprint_joint" type="fixed">
     <parent link="base_footprint"/>
     <child link="base_link"/>
-    <origin xyz="0 0 ${wheel_radius + base_height/2}" rpy="0 0 0"/>
+    <origin xyz="0 0 ${wheel_radius}" rpy="0 0 0"/>
   </joint>
-  <!-- ===================== CHASSIS (base_link) ===================== -->
   <link name="base_link">
     <visual>
@@ -39,5 +21,5 @@
       </geometry>
       <material name="blue">
-        <color rgba="0.0 0.2 0.8 1.0"/>
+        <color rgba="0.0 0.0 0.8 1.0"/>
       </material>
     </visual>
@@ -49,22 +31,14 @@
     <inertial>
       <mass value="5.0"/>
-      <!-- box inertia: Ixx = m(w²+h²)/12, etc. -->
-      <inertia
-        ixx="${5.0*(base_width*base_width + base_height*base_height)/12.0}"
-        ixy="0" ixz="0"
-        iyy="${5.0*(base_length*base_length + base_height*base_height)/12.0}"
-        iyz="0"
-        izz="${5.0*(base_length*base_length + base_width*base_width)/12.0}"/>
+      <!-- box: ixx=(m/12)(w²+h²), iyy=(m/12)(l²+h²), izz=(m/12)(l²+w²) -->
+      <inertia ixx="0.04688" ixy="0.0" ixz="0.0"
+               iyy="0.07604" iyz="0.0" izz="0.10417"/>
     </inertial>
   </link>
-  <!-- ===================== LEFT WHEEL (rear) ===================== -->
-  <!--
-    Joint z = -base_height/2  →  wheel centre in world = 0.145 - 0.075 = 0.07 = wheel_radius ✓
-  -->
+  <!-- ===================== LEFT WHEEL ===================== -->
   <joint name="left_wheel_joint" type="continuous">
     <parent link="base_link"/>
     <child link="left_wheel"/>
-    <origin xyz="${wheel_x} ${base_width/2 + wheel_width/2} ${-base_height/2}"
-            rpy="-1.5708 0 0"/>
+    <origin xyz="-0.05 ${base_width/2 + wheel_width/2} ${-base_height/2}" rpy="-1.5708 0 0"/>
     <axis xyz="0 0 1"/>
   </joint>
@@ -74,6 +48,6 @@
         <cylinder radius="${wheel_radius}" length="${wheel_width}"/>
       </geometry>
-      <material name="dark_gray">
-        <color rgba="0.15 0.15 0.15 1.0"/>
+      <material name="black">
+        <color rgba="0.0 0.0 0.0 1.0"/>
       </material>
     </visual>
@@ -84,20 +58,15 @@
     </collision>
     <inertial>
-      <mass value="0.8"/>
-      <!-- cylinder: Ixx=Iyy = m(3r²+h²)/12, Izz = mr²/2 -->
-      <inertia
-        ixx="${0.8*(3*wheel_radius*wheel_radius + wheel_width*wheel_width)/12.0}"
-        ixy="0" ixz="0"
-        iyy="${0.8*(3*wheel_radius*wheel_radius + wheel_width*wheel_width)/12.0}"
-        iyz="0"
-        izz="${0.8*wheel_radius*wheel_radius/2.0}"/>
+      <mass value="0.5"/>
+      <!-- cylinder: ixx=iyy=(m/12)(3r²+h²), izz=(m/2)r² -->
+      <inertia ixx="0.00038" ixy="0.0" ixz="0.0"
+               iyy="0.00038" iyz="0.0" izz="0.00063"/>
     </inertial>
   </link>
-  <!-- ===================== RIGHT WHEEL (rear) ===================== -->
+  <!-- ===================== RIGHT WHEEL ===================== -->
   <joint name="right_wheel_joint" type="continuous">
     <parent link="base_link"/>
     <child link="right_wheel"/>
-    <origin xyz="${wheel_x} ${-(base_width/2 + wheel_width/2)} ${-base_height/2}"
-            rpy="-1.5708 0 0"/>
+    <origin xyz="-0.05 ${-(base_width/2 + wheel_width/2)} ${-base_height/2}" rpy="-1.5708 0 0"/>
     <axis xyz="0 0 1"/>
   </joint>
@@ -107,5 +76,7 @@
         <cylinder radius="${wheel_radius}" length="${wheel_width}"/>
       </geometry>
-      <material name="dark_gray"/>
+      <material name="black">
+        <color rgba="0.0 0.0 0.0 1.0"/>
+      </material>
     </visual>
     <collision>
@@ -115,57 +86,45 @@
     </collision>
     <inertial>
-      <mass value="0.8"/>
-      <inertia
-        ixx="${0.8*(3*wheel_radius*wheel_radius + wheel_width*wheel_width)/12.0}"
-        ixy="0" ixz="0"
-        iyy="${0.8*(3*wheel_radius*wheel_radius + wheel_width*wheel_width)/12.0}"
-        iyz="0"
-        izz="${0.8*wheel_radius*wheel_radius/2.0}"/>
+      <mass value="0.5"/>
+      <!-- cylinder: ixx=iyy=(m/12)(3r²+h²), izz=(m/2)r² -->
+      <inertia ixx="0.00038" ixy="0.0" ixz="0.0"
+               iyy="0.00038" iyz="0.0" izz="0.00063"/>
     </inertial>
   </link>
-  <!-- ===================== FRONT CASTER ===================== -->
-  <!--
-    Caster sphere radius = wheel_radius/2 = 0.035.
-    Its centre must be at z = caster_radius above base_footprint.
-    Joint z (relative to base_link at 0.145) = caster_radius - (wheel_radius+base_height/2)
-             = 0.035 - 0.145 = -0.110
-    Equivalently: -(base_height/2 + wheel_radius/2) = -(0.075+0.035) = -0.110 ✓
-  -->
+  <!-- ===================== CASTER WHEEL ===================== -->
+  <!-- Fixed joint + near-zero friction sphere = ball-joint behaviour (SDF style) -->
   <joint name="caster_joint" type="fixed">
     <parent link="base_link"/>
     <child link="caster_wheel"/>
-    <origin xyz="${base_length/2 - 0.06} 0 ${-(base_height/2 + caster_radius)}" rpy="0 0 0"/>
+    <!-- Caster at FRONT (+X) so it resists forward tipping when braking.
+         z lowered by wheel_radius/2 so sphere bottom (r=0.025) is flush with ground. -->
+    <origin xyz="${base_length/2 - 0.05} 0 ${-base_height/2 - wheel_radius/2}" rpy="0 0 0"/>
   </joint>
   <link name="caster_wheel">
     <visual>
       <geometry>
-        <sphere radius="${caster_radius}"/>
+        <sphere radius="${wheel_radius/2}"/>
       </geometry>
-      <material name="green">
-        <color rgba="0.0 0.8 0.2 1.0"/>
+      <material name="gray">
+        <color rgba="0.5 0.5 0.5 1.0"/>
       </material>
     </visual>
     <collision>
       <geometry>
-        <sphere radius="${caster_radius}"/>
+        <sphere radius="${wheel_radius/2}"/>
       </geometry>
     </collision>
     <inertial>
-      <mass value="0.2"/>
-      <!-- sphere: I = 2mr²/5 -->
-      <inertia
-        ixx="${2*0.2*caster_radius*caster_radius/5.0}"
-        ixy="0" ixz="0"
-        iyy="${2*0.2*caster_radius*caster_radius/5.0}"
-        iyz="0"
-        izz="${2*0.2*caster_radius*caster_radius/5.0}"/>
+      <mass value="0.1"/>
+      <!-- sphere: ixx=iyy=izz=(2/5)mr² = 0.4*0.1*0.025² -->
+      <inertia ixx="0.000025" ixy="0.0" ixz="0.0"
+               iyy="0.000025" iyz="0.0" izz="0.000025"/>
     </inertial>
   </link>
   <!-- ===================== LIDAR ===================== -->
-  <!-- Sits on the chassis top, slightly toward the rear so the camera has a clear view ahead -->
   <joint name="lidar_joint" type="fixed">
     <parent link="base_link"/>
     <child link="lidar_link"/>
-    <origin xyz="-0.05 0 ${base_height/2 + 0.025}" rpy="0 0 0"/>
+    <origin xyz="0 0 ${base_height/2 + 0.05}" rpy="0 0 0"/>
   </joint>
   <link name="lidar_link">
@@ -185,18 +144,18 @@
     <inertial>
       <mass value="0.1"/>
-      <inertia ixx="0.0001" ixy="0" ixz="0"
-               iyy="0.0001" iyz="0" izz="0.0001"/>
+      <inertia ixx="0.0001" ixy="0.0" ixz="0.0"
+               iyy="0.0001" iyz="0.0" izz="0.0001"/>
     </inertial>
   </link>
-  <!-- ===================== CAMERA (front face) ===================== -->
+  <!-- ===================== CAMERA ===================== -->
   <joint name="camera_joint" type="fixed">
     <parent link="base_link"/>
     <child link="camera_link"/>
-    <origin xyz="${base_length/2} 0 0" rpy="0 0 0"/>
+    <origin xyz="${base_length/2} 0 ${base_height/2}" rpy="0 0 0"/>
   </joint>
   <link name="camera_link">
     <visual>
       <geometry>
-        <box size="0.02 0.06 0.04"/>
+        <box size="0.02 0.05 0.03"/>
       </geometry>
       <material name="green">
@@ -206,6 +165,6 @@
     <inertial>
       <mass value="0.05"/>
-      <inertia ixx="0.0001" ixy="0" ixz="0"
-               iyy="0.0001" iyz="0" izz="0.0001"/>
+      <inertia ixx="0.0001" ixy="0.0" ixz="0.0"
+               iyy="0.0001" iyz="0.0" izz="0.0001"/>
     </inertial>
   </link>
@@ -219,6 +178,6 @@
     <inertial>
       <mass value="0.01"/>
-      <inertia ixx="0.0001" ixy="0" ixz="0"
-               iyy="0.0001" iyz="0" izz="0.0001"/>
+      <inertia ixx="0.0001" ixy="0.0" ixz="0.0"
+               iyy="0.0001" iyz="0.0" izz="0.0001"/>
     </inertial>
   </link>
